File: hardware/kicad/Rotary_phone_SMD2/Rotary_phone_SMD2.kicad_pcb (KiCad board)
At the start: 2 copper layers, 100 x 50 mm, 77 parts, among them J2 PINHD_1x2_Male, J3 PINHD_1x2_Male, J4 PINHD_1x2_Male, J5 PINHD_1x3_Male, J6 RJ12, J7 RJ12, J8 Screw_Terminal_2_P5.00mm, U1 ME6211C33M5G-N, U2 ESP32-C6-WROOM-1, U3 USBLC6-2SC6, U4 ES8388, U5 AG1171, U6 AG1171

Commit message: Add network/web layer, milestone-3 prompt playback, and hardware fixes
Squashes a long bring-up/dev session into one checkpoint (going forward,
commits will be per-feature/fix as requested):

- WiFi (NVS + Kconfig credentials), NTP, in-RAM log ring buffer, SPIFFS-backed
  storage layer, and a web UI (status/log/recordings/dial-guide/settings)
  styled to match the original Pi Flask app.
- Dual-board Kconfig (SMD2/THT) with runtime codec_detect, ES8388 driver,
  status LED breathing during WiFi connect.
- Real SMD2 hardware bugs found and fixed: USB D+/D- swap, AG1171 Vin/Vout
  swap, SLIC PD polarity, ES8388 DAC mute-by-default, single-ADC-channel mono
  capture bodge-fixed to true stereo (RIN1 rewire) with a feedback-loop gain
  fix once both lines went live-duplex for the first time.
- Bring-up console: micamp, tonemon, record, play, capture/pulsemon rework.
- New `player` component + streaming storage read/write API (heap-safe for
  files too big to buffer) wired into ACT_OPERATOR_HELP/ACT_PLAY_CLIP; host
  tool (gen_prompt.py) to synthesize/convert prompt WAVs and upload them.
- SMD3 KiCad project checked in (schematic/PCB source only, not 3D exports).

Co-Authored-By: Claude Sonnet 5 <noreply@anthropic.com>
Parts:
- moved D8 5.01 mm to (135.2, 115.0)
- moved D11 0.35 mm to (129.8, 115.0)
Routing:
- net Net-(D12-A): track 0.00 -> 22.8 mm
- net Net-(D11-A): track 0.00 -> 10.1 mm
- net Net-(D11-K): track 0.00 -> 7.47 mm
Changed lines of the file:
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@@
 	(footprint "JLCImport:1N4007W_C18199088"
 		(layer "F.Cu")
-		(at 130.1 115.05 90)
+		(at 129.75 115.05 90)
 		(descr "-55℃~+150℃ 1A 1V@1A 1kV 2uA@1000V 30A Standalone SOD-123FL Diodes - General Purpose ROHS")
 		(tags "1N4007W C18199088 SOD-123FL_L2.7-W1.8-LS3.8-RD hongjiacheng")
@@
 	(footprint "JLCImport:1N4007W_C18199088"
 		(layer "F.Cu")
-		(at 134.5 110.05 -90)
+		(at 135.25 115 -90)
 		(descr "-55℃~+150℃ 1A 1V@1A 1kV 2uA@1000V 30A Standalone SOD-123FL Diodes - General Purpose ROHS")
 		(tags "1N4007W C18199088 SOD-123FL_L2.7-W1.8-LS3.8-RD hongjiacheng")
@@
 		(tags "RJ12 connector")
 		(property "Reference" "J7"
-			(at -1.66 -2.16 90)
+			(at 3.01 6.79 90)
 			(layer "F.SilkS")
 			(effects
@@
 	)
 	(via
-		(at 132.4 115.15)
+		(at 126.5 115.25)
 		(size 0.6)
 		(drill 0.3)
@@
 	)
 	(via
-		(at 137.5 115.35)
+		(at 136.75 116.75)
 		(size 0.6)
 		(drill 0.3)
@@
 	)
 	(via
-		(at 134.5 109.95)
+		(at 127 121)
 		(size 0.6)
 		(drill 0.3)
@@
 	)
 	(via
-		(at 122.2 119.95)
+		(at 116.5 121.25)
 		(size 0.6)
 		(drill 0.3)
@@
 	)
 	(via
-		(at 129.9 115.15)
+		(at 138.75 114)
 		(size 0.6)
 		(drill 0.3)
@@
 	)
 	(segment
+		(start 140 104.45)
+		(end 141.76 106.21)
+		(width 0.4)
+		(layer "F.Cu")
+		(net "Net-(D12-A)")
+	)
+	(segment
+		(start 141.76 106.21)
+		(end 141.76 107.719016)
+		(width 0.4)
+		(layer "F.Cu")
+		(net "Net-(D12-A)")
+	)
+	(segment
+		(start 136.114016 113.365)
+		(end 135.25 113.365)
+		(width 0.4)
+		(layer "F.Cu")
+		(net "Net-(D12-A)")
+	)
+	(segment
+		(start 132.5 113.415)
+		(end 135.2 113.415)
+		(width 0.4)
+		(layer "F.Cu")
+		(net "Net-(D12-A)")
+	)
+	(segment
+		(start 141.76 107.719016)
+		(end 136.114016 113.365)
+		(width 0.4)
+		(layer "F.Cu")
+		(net "Net-(D12-A)")
+	)
+	(segment
+		(start 135.2 113.415)
+		(end 135.25 113.365)
+		(width 0.4)
+		(layer "F.Cu")
+		(net "Net-(D12-A)")
+	)
+	(segment
+		(start 132.5 113.415)
+		(end 132.5 107.02)
+		(width 0.4)
+		(layer "F.Cu")
+		(net "Net-(D12-A)")
+	)
+	(segment
+		(start 132.5 107.02)
+		(end 131.93 106.45)
+		(width 0.4)
+		(layer "F.Cu")
+		(net "Net-(D12-A)")
+	)
+	(segment
+		(start 129.75 106.81)
+		(end 129.39 106.45)
+		(width 0.4)
+		(layer "F.Cu")
+		(net "Net-(D11-A)")
+	)
+	(segment
+		(start 137.46 105.72)
+		(end 134.635 105.72)
+		(width 0.4)
+		(layer "F.Cu")
+		(net "Net-(D11-A)")
+	)
+	(segment
+		(start 129.75 113.415)
+		(end 129.75 106.81)
+		(width 0.4)
+		(layer "F.Cu")
+		(net "Net-(D11-A)")
+	)
+	(segment
+		(start 134.635 105.72)
+		(end 134.5 105.585)
+		(width 0.4)
+		(layer "F.Cu")
+		(net "Net-(D11-A)")
+	)
+	(segment
 		(start 53.05 89.95)
 		(end 58.650003 95.550003)
@@
 	)
 	(segment
+		(start 132.5 118.15)
+		(end 130.8 119.85)
+		(width 0.4)
+		(layer "F.Cu")
+		(net "Net-(D11-K)")
+	)
+	(segment
+		(start 129.75 118.8)
+		(end 130.8 119.85)
+		(width 0.4)
+		(layer "F.Cu")
+		(net "Net-(D11-K)")
+	)
+	(segment
+		(start 129.75 116.685)
+		(end 129.75 118.8)
+		(width 0.4)
+		(layer "F.Cu")
+		(net "Net-(D11-K)")
+	)
+	(segment
+		(start 132.5 116.685)
+		(end 132.5 118.15)
+		(width 0.4)
+		(layer "F.Cu")
+		(net "Net-(D11-K)")
+	)
+	(segment

Commit message: kicad: consolidate custom footprints/3D/symbols into libraries/
Move all per-project Scott.pretty, JLCImport.pretty, .3dshapes, and
.kicad_sym files into a single shared kicad/libraries/ directory.
Rename "Scott" library to "Custom" throughout. Update fp-lib-table,
sym-lib-table, .kicad_pcb, and .kicad_sch files in all 6 board
projects to resolve Custom: and JLCImport: via ${KIPRJMOD}/../libraries/.

Also fixes broken 3D model paths (hardcoded /Users/... and
_restore_backup_ references in SMD3/SMD4/AR5 PCBs).

Generated with [Devin](https://devin.ai)

Co-Authored-By: Devin <158243242+devin-ai-integration[bot]@users.noreply.github.com>
Parts:
- U5, U6: footprint Scott:AG1171_SIL -> Custom:AG1171_SIL
Changed lines of the file:
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@@
 		)
 		(embedded_fonts no)
-		(model "${KIPRJMOD}/Scott.3dshapes/87180-062LF.step"
+		(model "${KIPRJMOD}/../libraries/Custom.3dshapes/87180-062LF.step"
 			(offset
 				(xyz 3.175 -8.9 0)
@@
 		)
 	)
-	(footprint "Scott:AG1171_SIL"
+	(footprint "Custom:AG1171_SIL"
 		(layer "F.Cu")
 		(at 100.7 107.99)
@@
 		)
 		(embedded_fonts no)
-		(model "${KIPRJMOD}/Scott.3dshapes/AG1171.step"
+		(model "${KIPRJMOD}/../libraries/Custom.3dshapes/AG1171.step"
 			(offset
 				(xyz 31.25 4.3 0)
@@
 		)
 		(embedded_fonts no)
-		(model "${KIPRJMOD}/JLCImport.3dshapes/1N4007W_C18199088.wrl"
+		(model "${KIPRJMOD}/../libraries/JLCImport.3dshapes/1N4007W_C18199088.wrl"
 			(offset
 				(xyz 0 0 -0.09)
@@
 		)
 		(embedded_fonts no)
-		(model "${KIPRJMOD}/JLCImport.3dshapes/TYPE-C_16PIN_2MD_073.wrl"
+		(model "${KIPRJMOD}/../libraries/JLCImport.3dshapes/TYPE-C_16PIN_2MD_073.wrl"
 			(offset
 				(xyz 0 -1.2 1.68)
@@
 		)
 		(embedded_fonts no)
-		(model "${KIPRJMOD}/JLCImport.3dshapes/TF-01A.wrl"
+		(model "${KIPRJMOD}/../libraries/JLCImport.3dshapes/TF-01A.wrl"
 			(offset
 				(xyz 0.002223 -5.10134 0.14732)
@@
 		)
 		(embedded_fonts no)
-		(model "${KIPRJMOD}/JLCImport.3dshapes/1N4148W_C81598.wrl"
+		(model "${KIPRJMOD}/../libraries/JLCImport.3dshapes/1N4148W_C81598.wrl"
 			(offset
 				(xyz 0 0 0)
@@
 		)
 		(embedded_fonts no)
-		(model "${KIPRJMOD}/JLCImport.3dshapes/1N4007W_C18199088.wrl"
+		(model "${KIPRJMOD}/../libraries/JLCImport.3dshapes/1N4007W_C18199088.wrl"
 			(offset
 				(xyz 0 0 -0.09)
@@
 		)
 		(embedded_fonts no)
-		(model "${KIPRJMOD}/JLCImport.3dshapes/1N4007W_C18199088.wrl"
+		(model "${KIPRJMOD}/../libraries/JLCImport.3dshapes/1N4007W_C18199088.wrl"
 			(offset
 				(xyz 0 0 -0.09)
@@
 		)
 		(embedded_fonts no)
-		(model "${KIPRJMOD}/JLCImport.3dshapes/1N4007W_C18199088.wrl"
+		(model "${KIPRJMOD}/../libraries/JLCImport.3dshapes/1N4007W_C18199088.wrl"
 			(offset
 				(xyz 0 0 -0.09)
@@
 		)
 	)
-	(footprint "Scott:AG1171_SIL"
+	(footprint "Custom:AG1171_SIL"
 		(layer "F.Cu")
 		(at 100.71 95.29)
@@
 		)
 		(embedded_fonts no)
-		(model "${KIPRJMOD}/Scott.3dshapes/AG1171.step"
+		(model "${KIPRJMOD}/../libraries/Custom.3dshapes/AG1171.step"
 			(offset
 				(xyz 31.25 4.3 0)
@@
 		)
 		(embedded_fonts no)
-		(model "${KIPRJMOD}/JLCImport.3dshapes/1N4007W_C18199088.wrl"
+		(model "${KIPRJMOD}/../libraries/JLCImport.3dshapes/1N4007W_C18199088.wrl"
 			(offset
 				(xyz 0 0 -0.09)
@@
 		)
 		(embedded_fonts no)
-		(model "${KIPRJMOD}/JLCImport.3dshapes/1N4007W_C18199088.wrl"
+		(model "${KIPRJMOD}/../libraries/JLCImport.3dshapes/1N4007W_C18199088.wrl"
 			(offset
 				(xyz 0 0 -0.09)
@@
 		)
 		(embedded_fonts no)
-		(model "${KIPRJMOD}/JLCImport.3dshapes/1N4007W_C18199088.wrl"
+		(model "${KIPRJMOD}/../libraries/JLCImport.3dshapes/1N4007W_C18199088.wrl"
 			(offset
 				(xyz 0 0 -0.09)
@@
 		)
 		(embedded_fonts no)
-		(model "${KIPRJMOD}/Scott.3dshapes/87180-062LF.step"
+		(model "${KIPRJMOD}/../libraries/Custom.3dshapes/87180-062LF.step"
 			(offset
 				(xyz 3.175 -8.9 0)
@@
 		)
 		(embedded_fonts no)
-		(model "${KIPRJMOD}/JLCImport.3dshapes/1N4148W_C81598.wrl"
+		(model "${KIPRJMOD}/../libraries/JLCImport.3dshapes/1N4148W_C81598.wrl"
 			(offset
 				(xyz 0 0 0)
@@
 		)
 		(embedded_fonts no)
-		(model "${KIPRJMOD}/JLCImport.3dshapes/1N4007W_C18199088.wrl"
+		(model "${KIPRJMOD}/../libraries/JLCImport.3dshapes/1N4007W_C18199088.wrl"
 			(offset
 				(xyz 0 0 -0.09)
