File: hardware/kicad/Rotary_phone_SMD4/Rotary_phone_SMD4.kicad_pcb (KiCad board)
At the start: 2 copper layers, 110 x 52 mm, 64 parts, among them J1 Barrel_Jack_PTH_Slot, J3 PINHD_1x2_Male, J4 PINHD_1x2_Male, J5 PINHD_2x4_Male, J7 PINHD_1x3_Male, J8 RJ12, J9 RJ12, U1 ESP32-C6-DevKitC-1, U2 ES8388, U3 AG1171, U4 AG1171

Commit message: README board photo, SD self-test heap fix, SMD5 KiCad project, doc path fixes
- README: SMD4 board photo (docs/pics/) and wording tweaks
- sdcard: self-test reuses one buffer for read-back (halves peak heap;
  256KB contiguous wasn't available on a busy single-line board)
- SMD5 defaults / firmware README: point at ANALOG_REDIAL_SMD5.md
- Add the Analog Redial 5 (SMD5) KiCad project (schematic, PCB, dual
  DevKitC footprints); SMD2/SMD4 KiCad project/PCB touch-ups

Co-Authored-By: Claude Opus 5.5 <noreply@anthropic.com>
Other:
- board text added: "470uF"
- board text added: "Analog Redial 4.0 Major Hack 2026/08"
- board text removed: "Analog Phone 4.0 Major Hack 2026/08"
Changed lines of the file:
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@@
 		)
 	)
-	(gr_text "Analog Phone 4.0\nMajor Hack\n2026/08"
+	(gr_text "470uF"
+		(at 82.25 76.75 0)
+		(layer "F.SilkS")
+		(effects
+			(font
+				(size 1 1)
+				(bold yes)
+			)
+			(justify left bottom)
+		)
+	)
+	(gr_text "470uF"
+		(at 93.25 76.5 0)
+		(layer "F.SilkS")
+		(effects
+			(font
+				(size 1 1)
+				(bold yes)
+			)
+			(justify left bottom)
+		)
+	)
+	(gr_text "Analog Redial 4.0\nMajor Hack\n2026/08"
 		(at 55.15 93.5 90)
 		(layer "F.SilkS")

Commit message: kicad: consolidate custom footprints/3D/symbols into libraries/
Move all per-project Scott.pretty, JLCImport.pretty, .3dshapes, and
.kicad_sym files into a single shared kicad/libraries/ directory.
Rename "Scott" library to "Custom" throughout. Update fp-lib-table,
sym-lib-table, .kicad_pcb, and .kicad_sch files in all 6 board
projects to resolve Custom: and JLCImport: via ${KIPRJMOD}/../libraries/.

Also fixes broken 3D model paths (hardcoded /Users/... and
_restore_backup_ references in SMD3/SMD4/AR5 PCBs).

Generated with [Devin](https://devin.ai)

Co-Authored-By: Devin <158243242+devin-ai-integration[bot]@users.noreply.github.com>
Parts:
- J8, J9: footprint Scott:RJ12_Amphenol_87180_Horizontal -> Custom:RJ12_Amphenol_87180_Horizontal
- U3, U4: footprint Scott:AG1171_SIL -> Custom:AG1171_SIL
Changed lines of the file:
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@@
 		)
 	)
-	(footprint "Scott:AG1171_SIL"
+	(footprint "Custom:AG1171_SIL"
 		(locked yes)
 		(layer "F.Cu")
@@
 		)
 		(embedded_fonts no)
-		(model "${KIPRJMOD}/Scott.3dshapes/AG1171.step"
+		(model "${KIPRJMOD}/../libraries/Custom.3dshapes/AG1171.step"
 			(offset
 				(xyz 31.25 4.3 0)
@@
 		)
 		(embedded_fonts no)
-		(model "${KIPRJMOD}/_restore_backup_2026-08-30T20-24-25-026/JLCImport.3dshapes/1N4007W_C18199088.step"
+		(model "${KIPRJMOD}/../libraries/JLCImport.3dshapes/1N4007W_C18199088.step"
 			(offset
 				(xyz 0 0 -0.09)
@@
 		)
 		(embedded_fonts no)
-		(model "${KIPRJMOD}/_restore_backup_2026-08-30T20-24-25-026/JLCImport.3dshapes/TF-01A.step"
+		(model "${KIPRJMOD}/../libraries/JLCImport.3dshapes/TF-01A.step"
 			(offset
 				(xyz 0.002223 -5.10134 0.14732)
@@
 		)
 	)
-	(footprint "Scott:RJ12_Amphenol_87180_Horizontal"
+	(footprint "Custom:RJ12_Amphenol_87180_Horizontal"
 		(layer "F.Cu")
 		(at 61.07 88.46)
@@
 		)
 		(embedded_fonts no)
-		(model "${KIPRJMOD}/Scott.3dshapes/87180-066LF.step"
+		(model "${KIPRJMOD}/../libraries/Custom.3dshapes/87180-066LF.step"
 			(offset
 				(xyz 0 0 0)
@@
 		)
 		(embedded_fonts no)
-		(model "${KIPRJMOD}/_restore_backup_2026-08-30T20-24-25-026/JLCImport.3dshapes/1N4148W_C81598.step"
+		(model "${KIPRJMOD}/../libraries/JLCImport.3dshapes/1N4148W_C81598.step"
 			(offset
 				(xyz 0 0 0)
@@
 		)
 		(embedded_fonts no)
-		(model "${KIPRJMOD}/_restore_backup_2026-08-30T20-24-25-026/JLCImport.3dshapes/1N4007W_C18199088.step"
+		(model "${KIPRJMOD}/../libraries/JLCImport.3dshapes/1N4007W_C18199088.step"
 			(offset
 				(xyz 0 0 -0.09)
@@
 		)
 		(embedded_fonts no)
-		(model "${KIPRJMOD}/_restore_backup_2026-08-30T20-24-25-026/JLCImport.3dshapes/1N4007W_C18199088.step"
+		(model "${KIPRJMOD}/../libraries/JLCImport.3dshapes/1N4007W_C18199088.step"
 			(offset
 				(xyz 0 0 -0.09)
@@
 		)
 		(embedded_fonts no)
-		(model "${KIPRJMOD}/_restore_backup_2026-08-30T20-24-25-026/JLCImport.3dshapes/1N4007W_C18199088.step"
+		(model "${KIPRJMOD}/../libraries/JLCImport.3dshapes/1N4007W_C18199088.step"
 			(offset
 				(xyz 0 0 -0.09)
@@
 		)
 	)
-	(footprint "Scott:AG1171_SIL"
+	(footprint "Custom:AG1171_SIL"
 		(locked yes)
 		(layer "F.Cu")
@@
 		)
 		(embedded_fonts no)
-		(model "${KIPRJMOD}/Scott.3dshapes/AG1171.step"
+		(model "${KIPRJMOD}/../libraries/Custom.3dshapes/AG1171.step"
 			(offset
 				(xyz 31.25 4.3 0)
@@
 		)
 		(embedded_fonts no)
-		(model "${KIPRJMOD}/_restore_backup_2026-08-30T20-24-25-026/JLCImport.3dshapes/1N4007W_C18199088.step"
+		(model "${KIPRJMOD}/../libraries/JLCImport.3dshapes/1N4007W_C18199088.step"
 			(offset
 				(xyz 0 0 -0.09)
@@
 		)
 		(embedded_fonts no)
-		(model "${KIPRJMOD}/_restore_backup_2026-08-30T20-24-25-026/JLCImport.3dshapes/1N4007W_C18199088.step"
+		(model "${KIPRJMOD}/../libraries/JLCImport.3dshapes/1N4007W_C18199088.step"
 			(offset
 				(xyz 0 0 -0.09)
@@
 		)
 		(embedded_fonts no)
-		(model "${KIPRJMOD}/_restore_backup_2026-08-30T20-24-25-026/JLCImport.3dshapes/1N4007W_C18199088.step"
+		(model "${KIPRJMOD}/../libraries/JLCImport.3dshapes/1N4007W_C18199088.step"
 			(offset
 				(xyz 0 0 -0.09)
@@
 		)
 	)
-	(footprint "Scott:RJ12_Amphenol_87180_Horizontal"
+	(footprint "Custom:RJ12_Amphenol_87180_Horizontal"
 		(layer "F.Cu")
 		(at 75.67 88.46)
@@
 		)
 		(embedded_fonts no)
-		(model "${KIPRJMOD}/Scott.3dshapes/87180-066LF.step"
+		(model "${KIPRJMOD}/../libraries/Custom.3dshapes/87180-066LF.step"
 			(offset
 				(xyz 0 0 0)
@@
 		)
 		(embedded_fonts no)
-		(model "${KIPRJMOD}/_restore_backup_2026-08-30T20-24-25-026/JLCImport.3dshapes/1N4148W_C81598.step"
+		(model "${KIPRJMOD}/../libraries/JLCImport.3dshapes/1N4148W_C81598.step"
 			(offset
 				(xyz 0 0 0)
@@
 		)
 		(embedded_fonts no)
-		(model "${KIPRJMOD}/_restore_backup_2026-08-30T20-24-25-026/JLCImport.3dshapes/1N4007W_C18199088.step"
+		(model "${KIPRJMOD}/../libraries/JLCImport.3dshapes/1N4007W_C18199088.step"
 			(offset
 				(xyz 0 0 -0.09)
