File: hardware/kicad/rotary_phone_gateway/rotary_phone_gateway.kicad_pcb (KiCad board)
At the start: 2 copper layers, 100 x 100.2 mm, 59 parts, among them J1 RJ12, J2 RJ12, J3 Conn_01x02_Pin, J4 PINHD_1x2_Male, J5 PINHD_1x2_Male, J7 PINHD_1x3_Male, Q1 BC846, Q2 BC846, U1 ESP32-C6-DevKitM-1_1, U2 WM8731, U3 MCP1700x-180xxMB, U4 AG1170, U5 AG1170

Commit message: kicad: consolidate custom footprints/3D/symbols into libraries/
Move all per-project Scott.pretty, JLCImport.pretty, .3dshapes, and
.kicad_sym files into a single shared kicad/libraries/ directory.
Rename "Scott" library to "Custom" throughout. Update fp-lib-table,
sym-lib-table, .kicad_pcb, and .kicad_sch files in all 6 board
projects to resolve Custom: and JLCImport: via ${KIPRJMOD}/../libraries/.

Also fixes broken 3D model paths (hardcoded /Users/... and
_restore_backup_ references in SMD3/SMD4/AR5 PCBs).

Generated with [Devin](https://devin.ai)

Co-Authored-By: Devin <158243242+devin-ai-integration[bot]@users.noreply.github.com>
Parts:
- U2: footprint Scott:WM8731_SSOP-28 -> Custom:WM8731_SSOP-28
- U4, U5: footprint Scott:AG1170_SIL -> Custom:AG1170_SIL
Changed lines of the file:
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@@
 		)
 	)
-	(footprint "Scott:AG1170_SIL"
+	(footprint "Custom:AG1170_SIL"
 		(layer "F.Cu")
 		(at 78.81 66.04)
@@
 		)
 	)
-	(footprint "Scott:AG1170_SIL"
+	(footprint "Custom:AG1170_SIL"
 		(locked yes)
 		(layer "F.Cu")
@@
 		)
 	)
-	(footprint "Scott:WM8731_SSOP-28"
+	(footprint "Custom:WM8731_SSOP-28"
 		(layer "F.Cu")
 		(at 118.275 94 -90)
