File: hardware/kicad/rotary_phone_gateway/rotary_phone_gateway.kicad_sch (KiCad schematic)
At the start: 55 parts, among them J1 RJ12, J2 RJ12, J3 Conn_01x02_Pin, J4 PINHD_1x2_Male, J5 PINHD_1x2_Male, J7 PINHD_1x3_Male, Q1 BC846, Q2 BC846, U1 ESP32-C6-DevKitM-1, U2 WM8731SEDS/V-ssop28, U3 MCP1700x-180xxMB, U4 AG1170, U5 AG1170

Commit message: kicad: consolidate custom footprints/3D/symbols into libraries/
Move all per-project Scott.pretty, JLCImport.pretty, .3dshapes, and
.kicad_sym files into a single shared kicad/libraries/ directory.
Rename "Scott" library to "Custom" throughout. Update fp-lib-table,
sym-lib-table, .kicad_pcb, and .kicad_sch files in all 6 board
projects to resolve Custom: and JLCImport: via ${KIPRJMOD}/../libraries/.

Also fixes broken 3D model paths (hardcoded /Users/... and
_restore_backup_ references in SMD3/SMD4/AR5 PCBs).

Generated with [Devin](https://devin.ai)

Co-Authored-By: Devin <158243242+devin-ai-integration[bot]@users.noreply.github.com>
Parts:
- U2: footprint Scott:WM8731_SSOP-28 -> Custom:WM8731_SSOP-28; symbol Scott_Symbol_Library:WM8731 -> Custom_Symbol_Library:WM8731
- U4, U5: footprint Scott:AG1170_SIL -> Custom:AG1170_SIL; symbol Scott_Symbol_Library:AG1170_SIL -> Custom_Symbol_Library:AG1170_SIL
Changed lines of the file:
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@@
 	)
 	(symbol
-		(lib_id "Scott_Symbol_Library:AG1170_SIL")
+		(lib_id "Custom_Symbol_Library:AG1170_SIL")
 		(at 204.47 172.72 180)
 		(unit 1)
@@
 			)
 		)
-		(property "Footprint" "Scott:AG1170_SIL"
+		(property "Footprint" "Custom:AG1170_SIL"
 			(at 204.47 172.72 0)
 			(hide yes)
@@
 	)
 	(symbol
-		(lib_id "Scott_Symbol_Library:AG1170_SIL")
+		(lib_id "Custom_Symbol_Library:AG1170_SIL")
 		(at 203.2 102.87 180)
 		(unit 1)
@@
 			)
 		)
-		(property "Footprint" "Scott:AG1170_SIL"
+		(property "Footprint" "Custom:AG1170_SIL"
 			(at 203.2 102.87 0)
 			(hide yes)
@@
 	)
 	(symbol
-		(lib_id "Scott_Symbol_Library:WM8731")
+		(lib_id "Custom_Symbol_Library:WM8731")
 		(at 143.51 88.9 0)
 		(unit 1)
@@
 			)
 		)
-		(property "Footprint" "Scott:WM8731_SSOP-28"
+		(property "Footprint" "Custom:WM8731_SSOP-28"
 			(at 143.51 88.9 0)
 			(hide yes)
