File: hardware/kicad/Analog Redial 5/Analog Redial 5.kicad_sch (KiCad schematic)
At the start: 75 parts, among them J1 Barrel_Jack_PTH_Slot, J2 PINHD_1x8_Male, J3 PINHD_1x2_Male, J4 PINHD_1x2_Male, J5 PINHD_2x4_Male, J7 PINHD_1x3_Male, J8 RJ12, J9 RJ12, U1 ESP32-C6-DevKitC-1, U2 ES8388, U3 AG1171, U4 AG1171, U5 XC6206P332MR

Commit message: Consolidate custom KiCad library; point all boards at it
Every custom symbol and footprint this project used to keep in
hardware/kicad/libraries/ (AG1170/AG1171 SIL, the Amphenol/RJ12
connectors, both ESP32-C6 DevKit footprints, WM8731) is now in one
personal library shared across all KiCad projects on this machine:
~/Documents/KiCad/Custom/ (Custom.kicad_sym + Custom.pretty), registered
in KiCad's global symbol/footprint tables under the nickname 'Custom'.
That library also folds in the Schaffner choke, Phoenix terminal, TE
relay and test-point footprints from the old Scott_Library.pretty, and
the BM64 module symbol/footprint from the separate BM64 library.

SMD2, SMD4 and SMD5 ('Analog Redial 5') all used the AG1171_SIL symbol
under a stale 'Custom_Symbol_Library' nickname that was never actually
registered anywhere live (only resolvable from each schematic's own
embedded symbol cache) -- renamed to 'Custom:AG1171_SIL' in all three
schematics to match the new global library's nickname, which footprint
references already used. Verified with kicad-cli: netlist export clean
on all three, PCB export unaffected.

SMD2's project-local sym-lib-table/fp-lib-table had their own
'Custom_Symbol_Library'/'Custom' entries pointing at the
now-superseded repo copy -- removed, so it falls through to the
global table like SMD4/SMD5 already did. SMD4 and SMD5 never had
project-local entries for these, so no table changes were needed
there beyond the rename.

The old repo copy moves to
archive/hardware/kicad-libraries-pre-consolidation/ rather than being
deleted, per the project's archive convention -- its README explains
what superseded it and what a fresh clone still gets (schematics/PCBs
embed their own symbol/footprint copies, so they still open, view,
and export Gerbers/BOM fine; only live library editing needs the
global Custom library now).

Not touched: the untracked 'Analog Redial v6' board (newer WIP, not
yet added to git) got the same nickname rename and had its own stale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
Parts:
- U3, U4: symbol Custom_Symbol_Library:AG1171_SIL -> Custom:AG1171_SIL
Changed lines of the file:
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@@
 	)
 	(symbol
-		(lib_id "Custom_Symbol_Library:AG1171_SIL")
+		(lib_id "Custom:AG1171_SIL")
 		(at 308.61 160.02 180)
 		(unit 1)
@@
 	)
 	(symbol
-		(lib_id "Custom_Symbol_Library:AG1171_SIL")
+		(lib_id "Custom:AG1171_SIL")
 		(at 307.34 87.63 180)
 		(unit 1)
