File: hardware/kicad/Old/Analog Redial v3/Analog Redial v3.kicad_sch (KiCad schematic)
At the start: 75 parts, among them J1 Barrel_Jack_PTH_Slot, J2 PINHD_1x8_Male, J3 PINHD_1x2_Male, J4 PINHD_1x2_Male, J5 PINHD_2x4_Male, J7 PINHD_1x3_Male, J8 RJ12, J9 RJ12, U1 ESP32-C6-DevKitC-1, U2 ES8388, U3 AG1171, U4 AG1171, U5 XC6206P332MR

Commit message: Rename KiCad projects to Analog Redial v2/v3/v4/v5
Rotary_phone_SMD2 -> "Analog Redial v2", Old/Rotary_phone_SMD3 ->
"Old/Analog Redial v3", Rotary_phone_SMD4 -> "Analog Redial v4", and
"Analog Redial 5" -> "Analog Redial v5": directories, project files, and the
project-name references inside them (schematic annotation instances, the
PCB's sheet-file fields), checked by exporting each netlist -- every part is
still annotated. Silkscreen text and the SMD2 Gerber outputs keep their
names. Doc and code references updated (link targets URL-encoded); two
already-broken SMD2 BOM CSV links fixed on the way.

Firmware board-type names (CONFIG_BOARD_TYPE_SMD2/SMD4/SMD5) unchanged.

Co-Authored-By: Claude Opus 5.5 <noreply@anthropic.com>
Parts:
- removed C22, C23, C24, C25, C26: 1uF, Capacitor_SMD:C_0402_1005Metric, symbol PCM_SparkFun-Capacitor:C_Small
- removed J2: PINHD_1x8_Male, Connector_PinHeader_2.54mm:PinHeader_1x08_P2.54mm_Vertical, symbol PCM_SL_Pin_Headers:PINHD_1x8_Male
- removed JP2, JP3: (no value), PCM_SparkFun-Jumper:Jumper_3_NC-1_Trace_NoSilk, symbol Jumper:SolderJumper_3_Bridged12
- removed R16: 1k, Resistor_SMD:R_0402_1005Metric, symbol PCM_SparkFun-Resistor:R
- removed R17: 100k, Resistor_SMD:R_0402_1005Metric, symbol PCM_SparkFun-Resistor:R
- removed U5: XC6206P332MR, Package_TO_SOT_SMD:SOT-23-3, symbol Regulator_Linear:XC6206PxxxMR
- added J2: PINHD_1x2_Male, Connector_PinHeader_2.54mm:PinHeader_1x02_P2.54mm_Vertical, symbol PCM_SL_Pin_Headers:PINHD_1x2_Male
- C10, C11: value 47uF -> 100uF; footprint Capacitor_THT:C_Disc_D4.7mm_W2.5mm_P5.00mm -> Capacitor_SMD:C_1206_3216Metric
- D10, D11, D4, D5, D6, D7, D8, D9: value SM4007PL -> 1N4007; footprint Diode_SMD:Nexperia_CFP3_SOD-123W -> JLCImport:1N4007W_C18199088
- R12, R14: value 100k -> 15k
- R8, R9: value 10k -> 8.2k
- U1: footprint Custom:ESP32-C6-DevKitC-dual -> PCM_Espressif:ESP32-C6-DevKitC-1
- U3, U4: symbol Custom:AG1171_SIL -> Custom_Symbol_Library:AG1171_SIL
Connections:
- net GND: now also J2.2
- net I2S_MCLK: now also U1.12 (GPIO2)
- net Xtra1: now reaches U1.13 (GPIO3)
- net Xtra1: now also J2.1
- net at U1.30 (GPIO17/U0RXD): now also J4.1
- net at U1.31 (GPIO16/U0TXD): now also J3.1
- net GPIO12: no longer names the net of U1.19 (GPIO12/USB_D-)
- net GPIO12: no longer J4.1
- net GPIO13: no longer names the net of U1.20 (GPIO13/USB_D+)
- net GPIO13: no longer J3.1
- net Line0Vin: no longer names the net of C12.2, U4.9 (Vin)
- net Line0Vout: no longer names the net of C13.2, U4.10 (Vout)
- net MFB: no longer names the net of U1.29 (GPIO15/JTAG)
- net SD_CD: no longer names the net of Card1.9 (CD)
Other:
- note added: "Fixes: 470 uF capacitors are 8mm/3.5 pitch add reset jumper Fix cross-wired usb D+/D- Connect redundant usb-c wires so cables work in both directions In/out audio lines were swapped! Change Line0/1 in/out to mic for better readability Move Ch2 mic from Lin2 to Rin1 to fix error Todo: cleaner routing for USB D+/D- ? Test use of single P6KE82"
- note added: "Line 1: Left"
- note added: "Line 2: Right"
- note added: "NC D+"
- note added: "NC D-"
- note added: "NC Jtag"
- note added: "Use as UART header or 2x GPIO"
- note removed: "Bluetooth BM64 header"
- note removed: "CF Card"
- note removed: "Changes for SMD4: capacitor silkscreen needs to show capacitance value and line silkscreen note to add jumpbers for 2nd AG1171 silkscreen note to only use uSD OR SLIC #2 increase capacitor clearance and update footprint clearance to AG1171 board New esp32-c6 wide version option. (big change) add cuttable jumpers to select correct pinout for wide/cheap esp32-c6 change SHK voltage divider so it's c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"
- note removed: "Line 0: Left"
- note removed: "Line 1: Right"
- note removed: "UART to bluetooth board"
- note removed: "pin 5&6 matching cap mic inputs"
- moved on the sheet: C1, Card1, H1, H2, H3, H4, R1, R2
