File: hardware/kicad/Analog Redial v2/Analog Redial v2.kicad_sch (KiCad schematic)
At the start: 79 parts, among them J2 PINHD_1x2_Male, J3 PINHD_1x2_Male, J4 PINHD_1x2_Male, J5 PINHD_1x3_Male, J6 RJ12, J7 RJ12, J8 Screw_Terminal_2_P5.00mm, U1 ME6211C33M5G-N, U2 ESP32-C6-WROOM-1, U3 USBLC6-2SC6, U4 ES8388, U5 AG1171, U6 AG1171

Commit message: KiCad: rename the Old/ projects, drop stray "ESP32 Phone" copies
Old/rotary_phone_gateway -> "Old/Analog Redial v1" (the through-hole board)
and Old/Rotary_phone_SMD_old -> "Old/Analog Redial v2 draft", with the
project-name references inside updated (netlists export with every part
annotated). Removes the leftover "ESP32 Phone.kicad_*" projects from the v2,
v1 and v2-draft folders. Includes the v2 schematic's comment edit and its
rename fix-ups.

Co-Authored-By: Claude Opus 5.5 <noreply@anthropic.com>
Other:
- note added: "ERROR: D+ / D- incorrectly swapped on this board. Need to fix!"
- note removed: "ERROR: D+ / D- swapped on previous board. Need to fix!"
