File: hardware/kicad/Old/Analog Redial v2 draft/Analog Redial v2 draft.kicad_pcb (KiCad board)
At the start: 2 copper layers, 100 x 100.2 mm, 59 parts, among them J1 RJ12, J2 RJ12, J3 Conn_01x02_Pin, J4 PINHD_1x2_Male, J5 PINHD_1x2_Male, J7 PINHD_1x3_Male, Q1 BC846, Q2 BC846, U1 ESP32-C6-DevKitM-1_1, U2 WM8731, U3 MCP1700x-180xxMB, U4 AG1170, U5 AG1170

Commit message: KiCad: rename the Old/ projects, drop stray "ESP32 Phone" copies
Old/rotary_phone_gateway -> "Old/Analog Redial v1" (the through-hole board)
and Old/Rotary_phone_SMD_old -> "Old/Analog Redial v2 draft", with the
project-name references inside updated (netlists export with every part
annotated). Removes the leftover "ESP32 Phone.kicad_*" projects from the v2,
v1 and v2-draft folders. Includes the v2 schematic's comment edit and its
rename fix-ups.

Co-Authored-By: Claude Opus 5.5 <noreply@anthropic.com>
Parts:
- C1, C10, C11, C12, C15, C16, C17, C18, C3, C4, C5, C9: footprint Capacitor_THT:C_Disc_D3.0mm_W1.6mm_P2.50mm -> Capacitor_SMD:C_0402_1005Metric
- C13, C14: footprint Capacitor_THT:CP_Radial_D6.3mm_P2.50mm -> Capacitor_SMD:CP_Elec_8x10.5
- C19, C20: footprint Capacitor_THT:C_Disc_D3.0mm_W1.6mm_P2.50mm -> Capacitor_SMD:CP_Elec_8x10.5
- C2, C6: footprint Capacitor_THT:CP_Radial_D5.0mm_P2.00mm -> Capacitor_SMD:C_0603_1608Metric
- C7, C8: footprint Capacitor_THT:CP_Radial_D6.3mm_P2.50mm -> Capacitor_SMD:CP_Elec_6.3x7.7
- D1, D2, D3, D4, D5, D6, D7, D9: value 1N4004 -> 1N4148W; footprint Diode_THT:D_DO-41_SOD81_P10.16mm_Horizontal -> Diode_SMD:D_SOD-123
- D10, D8: value D_Zener P6KE82 -> P6KE82A; footprint Diode_THT:D_DO-41_SOD81_P10.16mm_Horizontal -> Diode_SMD:D_SOD-123
- R1, R10, R11, R12, R2, R3, R4, R5, R6, R7, R8, R9: footprint Resistor_THT:R_Axial_DIN0207_L6.3mm_D2.5mm_P10.16mm_Horizontal -> Resistor_SMD:R_0402_1005Metric
- REF** (x4): footprint MountingHole:MountingHole_3.2mm_M3_Pad_TopBottom -> Resistor_SMD:R_0402_1005Metric
