File: hardware/kicad/Analog Redial v5/Analog Redial v5.kicad_pcb (KiCad board)
At the start: 2 copper layers, 115 x 52 mm, 76 parts, among them J1 Barrel_Jack_PTH_Slot, J2 PINHD_1x8_Male, J3 PINHD_1x2_Male, J4 PINHD_1x2_Male, J5 PINHD_2x4_Male, J7 PINHD_1x3_Male, J8 RJ12, J9 RJ12, U1 ESP32-C6-DevKitC-1, U2 ES8388, U3 AG1171, U4 AG1171, U5 XC6206PxxxMR

Commit message: BOM and v5 board updates; drop the old DigiKey cart CSV
Scott's edits: BOM notes for the 30-pin clone module (aimed at v5), a
shipping row, Bluetooth marked as v5, and the resolved "Open items" list
removed; the v5 PCB as sent to fab (plus its project-name rename fix-ups);
hardware/2026-07-02T230626.csv deleted.

Co-Authored-By: Claude Opus 5.5 <noreply@anthropic.com>
Other:
- board text added: "Analog Redial v5"
- board text removed: "Analog Redial 5"
