File: PayPhone/Payphone_v1/Payphone_v1.kicad_sch (KiCad schematic)
At the start: 87 parts, among them J1 JST_05, J2 Molex_26-60-4030, J3 Molex_26-60-4040, J6 PINHD_1x5_Male, J7 PINHD_1x2_Male, J8 PINHD_1x2_Male, J9 PINHD_1x2_Male, K1 G6S-2, Q2 2N7000, Q3 IRF630, Q4 2N7000, Q5 2N7000, Q6 2N3906, U1 MCP23008-xP, U2 MC34063AP, U3 UC3843AN, U4 ADS1115IDGS

Commit message: final schematic, updated for SMT components.
Parts:
- removed Cp: 100pF, Capacitor_THT:C_Disc_D5.0mm_W2.5mm_P5.00mm, symbol Device:C_Small
- removed Q2, Q4, Q5: 2N7000, Package_TO_SOT_THT:TO-92_Inline, symbol Transistor_FET:2N7000
- removed Q6: 2N3906, Package_TO_SOT_THT:TO-92_Inline, symbol Transistor_BJT:2N3906
- added Q1, Q4: 2N7002, Package_TO_SOT_SMD:SOT-23, symbol Transistor_FET:2N7002
- added Q2: MMBT3904, Package_TO_SOT_SMD:SOT-23, symbol Transistor_BJT:MMBT3904
- added Q5: MMBT3906, PCM_JLCPCB:Q_SOT-23, symbol PCM_JLCPCB-Transistors:PNP,MMBT3906
- C16, C17, C2, C3, C4, C6, C8: footprint Capacitor_THT:C_Disc_D5.0mm_W2.5mm_P5.00mm -> Capacitor_SMD:C_0805_2012Metric
- Cf1: renamed from Cf; footprint Capacitor_THT:C_Disc_D5.0mm_W2.5mm_P5.00mm -> Capacitor_SMD:C_0805_2012Metric
- Cslope1: renamed from Cslope; footprint Capacitor_THT:C_Disc_D5.0mm_W2.5mm_P5.00mm -> Capacitor_SMD:C_0805_2012Metric
- Ct1: renamed from Ct; footprint Capacitor_THT:C_Disc_D5.0mm_W2.5mm_P5.00mm -> Capacitor_SMD:C_0805_2012Metric
- Cvcc1: renamed from Cvcc; footprint Capacitor_THT:C_Disc_D5.0mm_W2.5mm_P5.00mm -> Capacitor_SMD:C_0805_2012Metric
- Cvref1: renamed from Cvref; footprint Capacitor_THT:C_Disc_D5.0mm_W2.5mm_P5.00mm -> Capacitor_SMD:C_0805_2012Metric
- Cz1: renamed from Cz; footprint Capacitor_THT:C_Rect_L7.2mm_W2.5mm_P5.00mm_FKS2_FKP2_MKS2_MKP2 -> Capacitor_SMD:C_0805_2012Metric
- D1: footprint Diode_THT:D_DO-41_SOD81_P10.16mm_Horizontal -> Diode_SMD:D_SOD-123
- D4: footprint Diode_THT:D_DO-35_SOD27_P7.62mm_Horizontal -> Diode_SMD:D_SOD-123
- J1, J6: now not fitted
- R1, R10, R13, R14, R17, R18, R19, R2, R20, R21, R22, R23, R24, R25, R3, R4, R5, R6, R7, R8, R9, Rfbb1, Rfbb2, Rfbb3, Rfbb4, Rfbt1, Rfbt2, Rfbt3: footprint Resistor_THT:R_Axial_DIN0207_L6.3mm_D2.5mm_P10.16mm_Horizontal -> Resistor_SMD:R_0805_2012Metric
- R12: value 68R -> 82R; footprint Resistor_THT:R_Axial_DIN0207_L6.3mm_D2.5mm_P10.16mm_Horizontal -> Resistor_SMD:R_0805_2012Metric
- R32: renamed from R15; footprint Resistor_THT:R_Axial_DIN0207_L6.3mm_D2.5mm_P10.16mm_Horizontal -> Resistor_SMD:R_0805_2012Metric
- R33: renamed from R16; footprint Resistor_THT:R_Axial_DIN0207_L6.3mm_D2.5mm_P10.16mm_Horizontal -> Resistor_SMD:R_0805_2012Metric
- Rbl1: renamed from Rbleed1; value 1M -> 47k; footprint Resistor_THT:R_Axial_DIN0207_L6.3mm_D2.5mm_P10.16mm_Horizontal -> Resistor_SMD:R_0805_2012Metric
- Rbl2: renamed from Rbleed2; value 1M -> 47k; footprint Resistor_THT:R_Axial_DIN0207_L6.3mm_D2.5mm_P10.16mm_Horizontal -> Resistor_SMD:R_0805_2012Metric
- Rbl3: renamed from Rbleed3; value 1M -> 47k; footprint Resistor_THT:R_Axial_DIN0207_L6.3mm_D2.5mm_P10.16mm_Horizontal -> Resistor_SMD:R_0805_2012Metric
- Rf1: renamed from Rf; footprint Resistor_THT:R_Axial_DIN0207_L6.3mm_D2.5mm_P10.16mm_Horizontal -> Resistor_SMD:R_0805_2012Metric
- Rg1: renamed from Rg; footprint Resistor_THT:R_Axial_DIN0207_L6.3mm_D2.5mm_P10.16mm_Horizontal -> Resistor_SMD:R_0805_2012Metric
- Rslope1: renamed from Rslope; footprint Resistor_THT:R_Axial_DIN0207_L6.3mm_D2.5mm_P10.16mm_Horizontal -> Resistor_SMD:R_0805_2012Metric
- Rz1: renamed from Rz; footprint Resistor_THT:R_Axial_DIN0207_L6.3mm_D2.5mm_P10.16mm_Horizontal -> Resistor_SMD:R_0805_2012Metric
- renumbered Dz to Dz1, Qa to Qa1, Rcs to Rcs1
Connections:
- net 20V: now also R23.1, Q5.2 (E); no longer R23.2
- net EN_HV: now also Q1.1 (G)
- net GND: now also Q1.2 (S), Q2.2 (E), Q4.2 (S)
- net Q2_G: now also Q2.1 (B)
- net Q4_D: now also Q4.3 (D)
- net Q4_G: now also Q4.1 (G)
- net Q6_B: now also R23.2, Q5.1 (B); no longer R23.1
- net Q6_C: now also Q5.3 (C)
- net RLY_COIL: now also Q2.3 (C)
- net at R14.2: now also Q1.3 (D)
Other:
- note added: "Needs 10V on gate"
- note added: "Rz Likely high. Verify"
- note added: "Short if not using ADC monitor"
- note removed: "RELAY"
- moved on the sheet: C1, C16, C17, D3, D4, D6, J2, K1, Q3, R20, R21, R22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
