File: PayPhone/Payphone_v1/Payphone_v1.kicad_pcb (KiCad board)
At the start: 2 copper layers, 85 parts, among them J1 JST_05, J2 Molex_26-60-4030, J3 Molex_26-60-4040, J6 PINHD_1x5_Male, J7 PINHD_1x2_Male, J8 PINHD_1x2_Male, J9 PINHD_1x2_Male, K1 G6S-2, Q1 2N7002, Q2 MMBT3904, Q3 IRF630, Q4 2N7002, U1 MCP23008-xP, U2 MC34063AP, U3 UC3843AN, U4 ADS1115IDGS

Commit message: Payphone coin board: parts placed in groups with routing notes; HV indicator LED (D7, lights above 24 V); +3V3 renamed VIO (host's I2C logic level) with JP1 VIO=5V; green debug LEDs for the coin lines and EN_HV/POL/FIRE; Rbl1-3 1M
Parts:
- added D5: BZT52C22, Diode_SMD:D_SOD-123, F.Cu at (195.2, 142.5)
- added D7: LED red, LED_SMD:LED_0805_2012Metric, F.Cu at (194.6, 145.7)
- added Q5: MMBT3906, Package_TO_SOT_SMD:SOT-23, F.Cu at (157.9, 88.5)
- added R27: 33k, Resistor_SMD:R_1206_3216Metric, F.Cu at (189.5, 142.5)
- added R28: 33k, Resistor_SMD:R_1206_3216Metric, F.Cu at (189.5, 145.8)
- Cvcc1: value 0.1uF -> 0.1uF 50V
- D1: value 1N5819 -> 1N5819HW
- D2: value UF4003 -> ES2D; footprint Diode_THT:D_DO-41_SOD81_P10.16mm_Horizontal -> Diode_SMD:D_SMA
- D3: value 1.5KE150A -> SMBJ130A; footprint Diode_THT:D_DO-201AD_P15.24mm_Horizontal -> Diode_SMD:D_SMB
- D4: value 1N4148 -> 1N4148W
- D6: value 12V -> BZT52C12; footprint Diode_THT:D_DO-41_SOD81_P10.16mm_Horizontal -> Diode_SMD:D_SOD-123
- Dz1: value 1N4744A 15V -> SMAZ15 (15V 1W); footprint Diode_THT:D_DO-41_SOD81_P10.16mm_Horizontal -> Diode_SMD:D_SMA
- L1: value 100uH -> 100uH 7447471101; footprint Inductor_THT:L_Radial_D10.0mm_P5.00mm_Fastron_07M -> Inductor_THT:L_Radial_D12.0mm_P5.00mm_Fastron_11P
- L2: value 220uH -> 220uH 7447471221; footprint Inductor_THT:L_Radial_D10.0mm_P5.00mm_Fastron_07M -> Inductor_THT:L_Radial_D12.0mm_P5.00mm_Fastron_11P
- Q3: value IRF630 -> STN4NF20L; footprint Package_TO_SOT_THT:TO-220-3_Vertical -> Package_TO_SOT_SMD:SOT-223-3_TabPin2
- R11: footprint Resistor_THT:R_Axial_DIN0309_L9.0mm_D3.2mm_P12.70mm_Horizontal -> Resistor_SMD:R_2512_6332Metric
- R26: value 10R 0.5W -> 10R; footprint Resistor_THT:R_Axial_DIN0309_L9.0mm_D3.2mm_P12.70mm_Horizontal -> Resistor_SMD:R_1206_3216Metric
- R32: value 1.17M -> 1.18M; footprint Resistor_SMD:R_0805_2012Metric -> Resistor_SMD:R_1206_3216Metric
- Rbl1, Rbl2, Rbl3: value 47k -> 150k; footprint Resistor_SMD:R_0805_2012Metric -> Resistor_SMD:R_1206_3216Metric
- Rcs1: footprint Resistor_THT:R_Axial_DIN0414_L11.9mm_D4.5mm_P15.24mm_Horizontal -> Resistor_SMD:R_2512_6332Metric
- Rfbt1, Rfbt2, Rfbt3: footprint Resistor_SMD:R_0805_2012Metric -> Resistor_SMD:R_1206_3216Metric
- U1: value MCP23008-xP -> MCP23008-E/SO; footprint Package_DIP:DIP-18_W7.62mm -> Package_SO:SOIC-18W_7.5x11.6mm_P1.27mm
- U2: value MC34063AP -> MC34063ADR2G; footprint Package_DIP:DIP-8_W7.62mm -> Package_SO:SOIC-8_3.9x4.9mm_P1.27mm
- U3: value UC3843AN -> UC3843BD1R2G; footprint Package_DIP:DIP-8_W7.62mm -> Package_SO:SOIC-8_3.9x4.9mm_P1.27mm
- moved Q1 231.0 mm to (28.9, 117.6)
- moved R11 217.3 mm to (30.1, 136.8), turned to 90 degrees
- moved J6 212.9 mm to (37.7, 86.4), turned to 180 degrees
- moved D1 206.7 mm to (51.7, 139.2), turned to 180 degrees
- moved C5 197.7 mm to (22.9, 128.4)
- moved U2 196.7 mm to (41.5, 132.0), turned to 180 degrees
- moved C6 189.8 mm to (34.3, 128.4), turned to 90 degrees
- moved J1 183.4 mm to (46.2, 86.4), turned to 90 degrees
- moved R1 177.5 mm to (24.7, 116.4), turned to 90 degrees
- moved R12 176.9 mm to (34.3, 136.2), turned to 90 degrees
- moved J9 176.2 mm to (81.3, 146.2), turned to 90 degrees
- moved C8 174.8 mm to (49.3, 131.4), turned to 90 degrees
- moved J8 171.1 mm to (81.3, 141.7), turned to 90 degrees
- moved R14 169.2 mm to (34.9, 117.6), turned to 180 degrees
- moved R13 167.3 mm to (39.1, 123.0)
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Connections:
- net /Q2_G renamed /Q2_B
- net /Q6_B renamed /Q5_B
- C6 pad 2: unconnected-(C6-Pad2) -> +5V
- R24 pad 1: /Q6_C -> /Q5_C
Other:
- board text added: "COIN ROUTING - C2-C4 at J3, then R7-R9, pull-ups R4-R6. - Slow logic: any route back to U1 pins 10-12."
- board text added: "COIN SWITCH INPUTS"
- board text added: "DANGER: UP TO 120 V DC C1 STAYS CHARGED UNTIL THE HV LED (D7) IS OUT"
- board text added: "FIRE DRIVER"
- board text added: "FIRE ROUTING - FIRE arrives as VIO logic (long is fine); the level shift is here, by Q3. - GATE3 (R24 / R25 / D6 -> Q3 gate): a few mm only. - Pulse loop: C1+ -> K1 -> J2 -> coin relay -> K1 -> Q3 -> R26 -> GND -> C1-. Keep compact; R26 GND via toward C1-. - ISENSE (R26 top) -> U4 AIN2 as a signal; add 100 nF at AIN2."
- board text added: "HV ROUTING - HV, HV_*, SW2, COIL_A/B, RETURN: HV net class, 1.0 mm clearance. Check the GND pour honours it. - R32 stays at HV: only its 3 V tap (AIN0) goes to U4. - D3 straight across C1. Rbl1-3 near C1. - Rfbt1-3 are HV class too: HV comes to Rfbt1, the FB end (Rfbt3) sits at U3."
- board text added: "HV SET (fit jumpers) none 52 V J9 60 V J8 78 V J7 87 V all 119 V"
- board text added: "LAYOUT NOTES (User.Comments: not fabricated) - 2 layers: top = parts + routing; bottom = one solid GND pour, short jumpers only. - One ground, no splits: close each power loop on top, then stitch to the plane. - Power flows left to right: J6 -> stage 1 -> stage 2 -> C1 -> K1 -> J2. - Each block is a KiCad group: drag it as a unit. No board outline yet."
- board text added: "LOGIC (VIO): I/O EXPANDER + ADC"
- board text added: "LOGIC ROUTING - I2C + power from J6/J1 straight to U1 and U4; no power currents through this area. - C16 at U1 pin 18, C17 at U4 pin 8 (VDD), each with its own GND via. - R33 / R19 / R17 = low ends of the ADC dividers, kept at U4. Add 10-100 nF from each AIN pin to GND here (not in the schematic yet). - POL, FIRE, EN_HV leave U1 pins 14-16 as plain VIO logic lines: long runs are fine, never paral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"
- board text added: "POL ROUTING - Q2, D4 at K1 coil pins 1/12. - K1 contacts are HV: HV (3, 8) and RETURN (5, 10) cross, so route one pair on the bottom layer."
- board text added: "POLARITY RELAY"
- board text added: "STAGE 1 ROUTING - Hot loop: U2 pin 1 (SwC) -> D1 -> C7/C9 -> GND -> U2 pin 2. Smallest possible, all on top. - Input: J6 +5V -> C5/C6 -> R11 -> U2 pin 7 / L1. Wide traces (1 mm+): ~1 A peaks. - SW1 (L1 / D1 anode / U2 pin 1): short, small copper. - C8 at pin 3; R13/R14 at the FB pin (pin 5). - Join C5-C15 and U2 pins 2/4 GND on top, then several vias. - 20V leaves from C9/C15 to stage 2 (L2, U3) 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"
- board text added: "STAGE 1: 5 V -> 20 V"
- board text added: "STAGE 2 ROUTING - Hot loop: Qa1 drain -> D2 -> C1+ ... C1- -> Rcs1 -> Qa1 source. Smallest possible. Consider a 100 nF 250 V ceramic from D2 cathode to Rcs1 GND (not in the schematic yet). - SW2 (Qa1 drain / L2 / D2 anode) swings 0-120 V: short, nothing parallel to it. - Gate: U3 OUT -> Rg1 -> Qa1 gate; Dz1 right at gate/source. - CS: separate (Kelvin) trace from Rcs1 top pad to Rf1; Cf1 at the U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"
- board text added: "STAGE 2: 20 V -> HV"
